File: mainboard/2layer/kicad/RAM_48.kicad_sch (KiCad schematic)
At the start: 82 parts, among them U24 MMN4116, U25 MMN4116, U26 MMN4116, U27 MMN4116, U28 MMN4116, U29 MMN4116, U30 MMN4116, U31 MMN4116, U41 74LS157, U43 MMN4116, U44 MMN4116, U45 MMN4116, U46 MMN4116, U47 MMN4116, U48 MMN4116, U49 MMN4116, U50 MMN4116, U58 74LS157, U62 MMN4116, U63 MMN4116, U64 MMN4116, U65 MMN4116, U66 MMN4116, U67 MMN4116, U68 MMN4116, U69 MMN4116

Commit message: Fixes for PCB DRC: trace clearance, footprints, board edges
Parts:
- JP11, JP12, JP13, JP14, JP15, JP16, JP17, JP18, JP19, JP28, JP29, JP30, JP31, JP32, JP33, JP34, JP35, JP36, JP37, JP38, JP39, JP40, JP41, JP42, JP43, JP44: footprint Jumper:SolderJumper-2_P1.3mm_Open_TrianglePad1.0x1.5mm -> Cobra_original:SolderJumper-2_P1.3mm_Open_TrianglePad1.0x1.5mm
Changed lines of the file:
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@@
       (effects (font (size 1.27 1.27)) hide)
     )
-    (property "Footprint" "Jumper:SolderJumper-2_P1.3mm_Open_TrianglePad1.0x1.5mm" (at 177.165 184.15 0)
+    (property "Footprint" "Cobra_original:SolderJumper-2_P1.3mm_Open_TrianglePad1.0x1.5mm" (at 177.165 184.15 0)
       (effects (font (size 1.27 1.27)) hide)
     )
@@
       (effects (font (size 1.27 1.27)) hide)
     )
-    (property "Footprint" "Jumper:SolderJumper-2_P1.3mm_Open_TrianglePad1.0x1.5mm" (at 111.125 212.09 0)
+    (property "Footprint" "Cobra_original:SolderJumper-2_P1.3mm_Open_TrianglePad1.0x1.5mm" (at 111.125 212.09 0)
       (effects (font (size 1.27 1.27)) hide)
     )
@@
       (effects (font (size 1.27 1.27)) hide)
     )
-    (property "Footprint" "Jumper:SolderJumper-2_P1.3mm_Open_TrianglePad1.0x1.5mm" (at 144.145 240.03 0)
+    (property "Footprint" "Cobra_original:SolderJumper-2_P1.3mm_Open_TrianglePad1.0x1.5mm" (at 144.145 240.03 0)
       (effects (font (size 1.27 1.27)) hide)
     )
@@
       (effects (font (size 1.27 1.27)) hide)
     )
-    (property "Footprint" "Jumper:SolderJumper-2_P1.3mm_Open_TrianglePad1.0x1.5mm" (at 177.165 44.45 0)
+    (property "Footprint" "Cobra_original:SolderJumper-2_P1.3mm_Open_TrianglePad1.0x1.5mm" (at 177.165 44.45 0)
       (effects (font (size 1.27 1.27)) hide)
     )
@@
       (effects (font (size 1.27 1.27)) hide)
     )
-    (property "Footprint" "Jumper:SolderJumper-2_P1.3mm_Open_TrianglePad1.0x1.5mm" (at 177.165 156.21 0)
+    (property "Footprint" "Cobra_original:SolderJumper-2_P1.3mm_Open_TrianglePad1.0x1.5mm" (at 177.165 156.21 0)
       (effects (font (size 1.27 1.27)) hide)
     )
@@
       (effects (font (size 1.27 1.27)) hide)
     )
-    (property "Footprint" "Jumper:SolderJumper-2_P1.3mm_Open_TrianglePad1.0x1.5mm" (at 111.125 156.21 0)
+    (property "Footprint" "Cobra_original:SolderJumper-2_P1.3mm_Open_TrianglePad1.0x1.5mm" (at 111.125 156.21 0)
       (effects (font (size 1.27 1.27)) hide)
     )
@@
       (effects (font (size 1.27 1.27)) hide)
     )
-    (property "Footprint" "Jumper:SolderJumper-2_P1.3mm_Open_TrianglePad1.0x1.5mm" (at 144.145 156.21 0)
+    (property "Footprint" "Cobra_original:SolderJumper-2_P1.3mm_Open_TrianglePad1.0x1.5mm" (at 144.145 156.21 0)
       (effects (font (size 1.27 1.27)) hide)
     )
@@
       (effects (font (size 1.27 1.27)) hide)
     )
-    (property "Footprint" "Jumper:SolderJumper-2_P1.3mm_Open_TrianglePad1.0x1.5mm" (at 33.02 201.295 0)
+    (property "Footprint" "Cobra_original:SolderJumper-2_P1.3mm_Open_TrianglePad1.0x1.5mm" (at 33.02 201.295 0)
       (effects (font (size 1.27 1.27)) hide)
     )
@@
       (effects (font (size 1.27 1.27)) hide)
     )
-    (property "Footprint" "Jumper:SolderJumper-2_P1.3mm_Open_TrianglePad1.0x1.5mm" (at 143.51 128.27 0)
+    (property "Footprint" "Cobra_original:SolderJumper-2_P1.3mm_Open_TrianglePad1.0x1.5mm" (at 143.51 128.27 0)
       (effects (font (size 1.27 1.27)) hide)
     )
@@
       (effects (font (size 1.27 1.27)) hide)
     )
-    (property "Footprint" "Jumper:SolderJumper-2_P1.3mm_Open_TrianglePad1.0x1.5mm" (at 111.125 100.33 0)
+    (property "Footprint" "Cobra_original:SolderJumper-2_P1.3mm_Open_TrianglePad1.0x1.5mm" (at 111.125 100.33 0)
       (effects (font (size 1.27 1.27)) hide)
     )
@@
       (effects (font (size 1.27 1.27)) hide)
     )
-    (property "Footprint" "Jumper:SolderJumper-2_P1.3mm_Open_TrianglePad1.0x1.5mm" (at 111.125 44.45 0)
+    (property "Footprint" "Cobra_original:SolderJumper-2_P1.3mm_Open_TrianglePad1.0x1.5mm" (at 111.125 44.45 0)
       (effects (font (size 1.27 1.27)) hide)
     )
@@
       (effects (font (size 1.27 1.27)) hide)
     )
-    (property "Footprint" "Jumper:SolderJumper-2_P1.3mm_Open_TrianglePad1.0x1.5mm" (at 177.165 72.39 0)
+    (property "Footprint" "Cobra_original:SolderJumper-2_P1.3mm_Open_TrianglePad1.0x1.5mm" (at 177.165 72.39 0)
       (effects (font (size 1.27 1.27)) hide)
     )
@@
       (effects (font (size 1.27 1.27)) hide)
     )
-    (property "Footprint" "Jumper:SolderJumper-2_P1.3mm_Open_TrianglePad1.0x1.5mm" (at 144.145 212.09 0)
+    (property "Footprint" "Cobra_original:SolderJumper-2_P1.3mm_Open_TrianglePad1.0x1.5mm" (at 144.145 212.09 0)
       (effects (font (size 1.27 1.27)) hide)
     )
@@
       (effects (font (size 1.27 1.27)) hide)
     )
-    (property "Footprint" "Jumper:SolderJumper-2_P1.3mm_Open_TrianglePad1.0x1.5mm" (at 111.125 128.27 0)
+    (property "Footprint" "Cobra_original:SolderJumper-2_P1.3mm_Open_TrianglePad1.0x1.5mm" (at 111.125 128.27 0)
       (effects (font (size 1.27 1.27)) hide)
     )
@@
       (effects (font (size 1.27 1.27)) hide)
     )
-    (property "Footprint" "Jumper:SolderJumper-2_P1.3mm_Open_TrianglePad1.0x1.5mm" (at 176.53 100.33 0)
+    (property "Footprint" "Cobra_original:SolderJumper-2_P1.3mm_Open_TrianglePad1.0x1.5mm" (at 176.53 100.33 0)
       (effects (font (size 1.27 1.27)) hide)
     )
@@
       (effects (font (size 1.27 1.27)) hide)
     )
-    (property "Footprint" "Jumper:SolderJumper-2_P1.3mm_Open_TrianglePad1.0x1.5mm" (at 111.125 72.39 0)
+    (property "Footprint" "Cobra_original:SolderJumper-2_P1.3mm_Open_TrianglePad1.0x1.5mm" (at 111.125 72.39 0)
       (effects (font (size 1.27 1.27)) hide)
     )
@@
       (effects (font (size 1.27 1.27)) hide)
     )
-    (property "Footprint" "Jumper:SolderJumper-2_P1.3mm_Open_TrianglePad1.0x1.5mm" (at 111.125 184.15 0)
+    (property "Footprint" "Cobra_original:SolderJumper-2_P1.3mm_Open_TrianglePad1.0x1.5mm" (at 111.125 184.15 0)
       (effects (font (size 1.27 1.27)) hide)
     )
@@
       (effects (font (size 1.27 1.27)) hide)
     )
-    (property "Footprint" "Jumper:SolderJumper-2_P1.3mm_Open_TrianglePad1.0x1.5mm" (at 144.145 72.39 0)
+    (property "Footprint" "Cobra_original:SolderJumper-2_P1.3mm_Open_TrianglePad1.0x1.5mm" (at 144.145 72.39 0)
       (effects (font (size 1.27 1.27)) hide)
     )
@@
       (effects (font (size 1.27 1.27)) hide)
     )
-    (property "Footprint" "Jumper:SolderJumper-2_P1.3mm_Open_TrianglePad1.0x1.5mm" (at 177.165 212.09 0)
+    (property "Footprint" "Cobra_original:SolderJumper-2_P1.3mm_Open_TrianglePad1.0x1.5mm" (at 177.165 212.09 0)
       (effects (font (size 1.27 1.27)) hide)
     )
@@
       (effects (font (size 1.27 1.27)) hide)
     )
-    (property "Footprint" "Jumper:SolderJumper-2_P1.3mm_Open_TrianglePad1.0x1.5mm" (at 111.125 240.03 0)
+    (property "Footprint" "Cobra_original:SolderJumper-2_P1.3mm_Open_TrianglePad1.0x1.5mm" (at 111.125 240.03 0)
       (effects (font (size 1.27 1.27)) hide)
     )
@@
       (effects (font (size 1.27 1.27)) hide)
     )
-    (property "Footprint" "Jumper:SolderJumper-2_P1.3mm_Open_TrianglePad1.0x1.5mm" (at 177.165 240.03 0)
+    (property "Footprint" "Cobra_original:SolderJumper-2_P1.3mm_Open_TrianglePad1.0x1.5mm" (at 177.165 240.03 0)
       (effects (font (size 1.27 1.27)) hide)
     )
@@
       (effects (font (size 1.27 1.27)) hide)
     )
-    (property "Footprint" "Jumper:SolderJumper-2_P1.3mm_Open_TrianglePad1.0x1.5mm" (at 144.145 44.45 0)
+    (property "Footprint" "Cobra_original:SolderJumper-2_P1.3mm_Open_TrianglePad1.0x1.5mm" (at 144.145 44.45 0)
       (effects (font (size 1.27 1.27)) hide)
     )
@@
       (effects (font (size 1.27 1.27)) hide)
     )
-    (property "Footprint" "Jumper:SolderJumper-2_P1.3mm_Open_TrianglePad1.0x1.5mm" (at 176.53 128.27 0)
+    (property "Footprint" "Cobra_original:SolderJumper-2_P1.3mm_Open_TrianglePad1.0x1.5mm" (at 176.53 128.27 0)
       (effects (font (size 1.27 1.27)) hide)
     )
@@
       (effects (font (size 1.27 1.27)) hide)
     )
-    (property "Footprint" "Jumper:SolderJumper-2_P1.3mm_Open_TrianglePad1.0x1.5mm" (at 33.02 212.09 0)
+    (property "Footprint" "Cobra_original:SolderJumper-2_P1.3mm_Open_TrianglePad1.0x1.5mm" (at 33.02 212.09 0)
       (effects (font (size 1.27 1.27)) hide)
     )
@@
       (effects (font (size 1.27 1.27)) hide)
     )
-    (property "Footprint" "Jumper:SolderJumper-2_P1.3mm_Open_TrianglePad1.0x1.5mm" (at 143.51 100.33 0)
+    (property "Footprint" "Cobra_original:SolderJumper-2_P1.3mm_Open_TrianglePad1.0x1.5mm" (at 143.51 100.33 0)
       (effects (font (size 1.27 1.27)) hide)
     )
@@
       (effects (font (size 1.27 1.27)) hide)
     )
-    (property "Footprint" "Jumper:SolderJumper-2_P1.3mm_Open_TrianglePad1.0x1.5mm" (at 144.145 184.15 0)
-      (effects (font (size 1.27 1.27)) hide)
-    )
+    (property "Footprint" "Cobra_original:SolderJumper-2_P1.3mm_Open_TrianglePad1.0x1.5mm" (at 144.145 184.15 0)
+      (effects (font (size 1.27 1.27)) hide)
+    )
