File: mainboard/2layer/kicad/Video_memory.kicad_sch (KiCad schematic)
At the start: 43 parts, among them U10 MMN4116, U11 MMN4116, U4 MMN4116, U5 MMN4116, U6 MMN4116, U7 MMN4116, U76 P8212, U8 MMN4116, U9 MMN4116

Commit message: Fix resistor values on video memory page
Parts:
- R20, R22, R23: value 33 -> 1K
Changed lines of the file:
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@@
       (effects (font (size 1.27 1.27)))
     )
-    (property "Value" "33" (at 124.46 50.8 90)
-      (effects (font (size 1.27 1.27)) hide)
+    (property "Value" "33" (at 129.54 52.07 90)
+      (effects (font (size 1.27 1.27)))
     )
     (property "Footprint" "Cobra_original:R_Axial_DIN0204_L3.6mm_D1.6mm_P5.08mm_Horizontal" (at 129.54 52.07 0)
@@
       (effects (font (size 1.27 1.27)))
     )
-    (property "Value" "33" (at 124.46 53.34 90)
-      (effects (font (size 1.27 1.27)) hide)
+    (property "Value" "33" (at 129.54 54.61 90)
+      (effects (font (size 1.27 1.27)))
     )
     (property "Footprint" "Cobra_original:R_Axial_DIN0204_L3.6mm_D1.6mm_P5.08mm_Horizontal" (at 129.54 54.61 0)
@@
       (effects (font (size 1.27 1.27)))
     )
-    (property "Value" "33" (at 124.46 55.88 90)
-      (effects (font (size 1.27 1.27)) hide)
+    (property "Value" "33" (at 129.54 57.15 90)
+      (effects (font (size 1.27 1.27)))
     )
     (property "Footprint" "Cobra_original:R_Axial_DIN0204_L3.6mm_D1.6mm_P5.08mm_Horizontal" (at 129.54 57.15 0)
@@
       (effects (font (size 1.27 1.27)))
     )
-    (property "Value" "33" (at 134.62 58.42 90)
-      (effects (font (size 1.27 1.27)) hide)
+    (property "Value" "33" (at 129.54 59.69 90)
+      (effects (font (size 1.27 1.27)))
     )
     (property "Footprint" "Cobra_original:R_Axial_DIN0204_L3.6mm_D1.6mm_P5.08mm_Horizontal" (at 129.54 59.69 0)
@@
       (effects (font (size 1.27 1.27)))
     )
-    (property "Value" "33" (at 134.62 60.96 90)
-      (effects (font (size 1.27 1.27)) hide)
+    (property "Value" "33" (at 129.54 62.23 90)
+      (effects (font (size 1.27 1.27)))
     )
     (property "Footprint" "Cobra_original:R_Axial_DIN0204_L3.6mm_D1.6mm_P5.08mm_Horizontal" (at 129.54 62.23 0)
@@
       (effects (font (size 1.27 1.27)))
     )
-    (property "Value" "33" (at 134.62 63.5 90)
-      (effects (font (size 1.27 1.27)) hide)
+    (property "Value" "33" (at 129.54 64.77 90)
+      (effects (font (size 1.27 1.27)))
     )
     (property "Footprint" "Cobra_original:R_Axial_DIN0204_L3.6mm_D1.6mm_P5.08mm_Horizontal" (at 129.54 64.77 0)
@@
       (effects (font (size 1.27 1.27)))
     )
-    (property "Value" "33" (at 134.62 66.04 90)
-      (effects (font (size 1.27 1.27)) hide)
+    (property "Value" "33" (at 129.54 67.31 90)
+      (effects (font (size 1.27 1.27)))
     )
     (property "Footprint" "Cobra_original:R_Axial_DIN0204_L3.6mm_D1.6mm_P5.08mm_Horizontal" (at 129.54 67.31 0)
@@
       (effects (font (size 1.27 1.27)))
     )
-    (property "Value" "33" (at 134.62 73.66 90)
-      (effects (font (size 1.27 1.27)) hide)
+    (property "Value" "33" (at 129.54 74.93 90)
+      (effects (font (size 1.27 1.27)))
     )
     (property "Footprint" "Cobra_original:R_Axial_DIN0204_L3.6mm_D1.6mm_P5.08mm_Horizontal" (at 129.54 74.93 0)
@@
       (effects (font (size 1.27 1.27)))
     )
-    (property "Value" "33" (at 134.62 76.2 90)
-      (effects (font (size 1.27 1.27)) hide)
+    (property "Value" "33" (at 129.54 77.47 90)
+      (effects (font (size 1.27 1.27)))
     )
     (property "Footprint" "Cobra_original:R_Axial_DIN0204_L3.6mm_D1.6mm_P5.08mm_Horizontal" (at 129.54 77.47 0)
@@
       (effects (font (size 1.27 1.27)))
     )
-    (property "Value" "33" (at 134.62 78.74 90)
-      (effects (font (size 1.27 1.27)) hide)
+    (property "Value" "33" (at 129.54 80.01 90)
+      (effects (font (size 1.27 1.27)))
     )
     (property "Footprint" "Cobra_original:R_Axial_DIN0204_L3.6mm_D1.6mm_P5.08mm_Horizontal" (at 129.54 80.01 0)
@@
       (effects (font (size 1.27 1.27)))
     )
-    (property "Value" "33" (at 134.62 87.63 90)
-      (effects (font (size 1.27 1.27)) hide)
+    (property "Value" "1K" (at 129.54 88.9 90)
+      (effects (font (size 1.27 1.27)))
     )
     (property "Footprint" "Cobra_original:R_Axial_DIN0204_L3.6mm_D1.6mm_P5.08mm_Horizontal" (at 129.54 88.9 0)
@@
       (effects (font (size 1.27 1.27)))
     )
-    (property "Value" "33" (at 134.62 90.17 90)
-      (effects (font (size 1.27 1.27)) hide)
+    (property "Value" "1K" (at 129.54 91.44 90)
+      (effects (font (size 1.27 1.27)))
     )
     (property "Footprint" "Cobra_original:R_Axial_DIN0204_L3.6mm_D1.6mm_P5.08mm_Horizontal" (at 129.54 91.44 0)
@@
       (effects (font (size 1.27 1.27)))
     )
-    (property "Value" "33" (at 134.62 92.71 90)
-      (effects (font (size 1.27 1.27)) hide)
+    (property "Value" "1K" (at 129.54 93.98 90)
+      (effects (font (size 1.27 1.27)))
     )
     (property "Footprint" "Cobra_original:R_Axial_DIN0204_L3.6mm_D1.6mm_P5.08mm_Horizontal" (at 129.54 93.98 0)

Commit message: Fixes for PCB DRC: trace clearance, footprints, board edges
Parts:
- JP14: footprint Jumper:SolderJumper-2_P1.3mm_Open_TrianglePad1.0x1.5mm -> Cobra_original:SolderJumper-2_P1.3mm_Open_TrianglePad1.0x1.5mm
Changed lines of the file:
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@@
       (effects (font (size 1.27 1.27)) hide)
     )
-    (property "Footprint" "Jumper:SolderJumper-2_P1.3mm_Open_TrianglePad1.0x1.5mm" (at 50.165 134.62 0)
+    (property "Footprint" "Cobra_original:SolderJumper-2_P1.3mm_Open_TrianglePad1.0x1.5mm" (at 50.165 134.62 0)
       (effects (font (size 1.27 1.27)) hide)
     )
@@
       (effects (font (size 1.27 1.27)) hide)
     )
-    (property "Footprint" "Jumper:SolderJumper-2_P1.3mm_Open_TrianglePad1.0x1.5mm" (at 50.165 218.44 0)
+    (property "Footprint" "Cobra_original:SolderJumper-2_P1.3mm_Open_TrianglePad1.0x1.5mm" (at 50.165 218.44 0)
       (effects (font (size 1.27 1.27)) hide)
     )
@@
       (effects (font (size 1.27 1.27)) hide)
     )
-    (property "Footprint" "Jumper:SolderJumper-2_P1.3mm_Open_TrianglePad1.0x1.5mm" (at 50.165 78.74 0)
+    (property "Footprint" "Cobra_original:SolderJumper-2_P1.3mm_Open_TrianglePad1.0x1.5mm" (at 50.165 78.74 0)
       (effects (font (size 1.27 1.27)) hide)
     )
@@
       (effects (font (size 1.27 1.27)) hide)
     )
-    (property "Footprint" "Jumper:SolderJumper-2_P1.3mm_Open_TrianglePad1.0x1.5mm" (at 50.165 190.5 0)
+    (property "Footprint" "Cobra_original:SolderJumper-2_P1.3mm_Open_TrianglePad1.0x1.5mm" (at 50.165 190.5 0)
       (effects (font (size 1.27 1.27)) hide)
     )
@@
       (effects (font (size 1.27 1.27)) hide)
     )
-    (property "Footprint" "Jumper:SolderJumper-2_P1.3mm_Open_TrianglePad1.0x1.5mm" (at 50.165 246.38 0)
+    (property "Footprint" "Cobra_original:SolderJumper-2_P1.3mm_Open_TrianglePad1.0x1.5mm" (at 50.165 246.38 0)
       (effects (font (size 1.27 1.27)) hide)
     )
@@
       (effects (font (size 1.27 1.27)) hide)
     )
-    (property "Footprint" "Jumper:SolderJumper-2_P1.3mm_Open_TrianglePad1.0x1.5mm" (at 50.165 106.68 0)
+    (property "Footprint" "Cobra_original:SolderJumper-2_P1.3mm_Open_TrianglePad1.0x1.5mm" (at 50.165 106.68 0)
       (effects (font (size 1.27 1.27)) hide)
     )
@@
       (effects (font (size 1.27 1.27)) hide)
     )
-    (property "Footprint" "Jumper:SolderJumper-2_P1.3mm_Open_TrianglePad1.0x1.5mm" (at 50.165 50.8 0)
+    (property "Footprint" "Cobra_original:SolderJumper-2_P1.3mm_Open_TrianglePad1.0x1.5mm" (at 50.165 50.8 0)
       (effects (font (size 1.27 1.27)) hide)
     )
@@
       (effects (font (size 1.27 1.27)) hide)
     )
-    (property "Footprint" "Jumper:SolderJumper-2_P1.3mm_Open_TrianglePad1.0x1.5mm" (at 50.165 162.56 0)
-      (effects (font (size 1.27 1.27)) hide)
-    )
+    (property "Footprint" "Cobra_original:SolderJumper-2_P1.3mm_Open_TrianglePad1.0x1.5mm" (at 50.165 162.56 0)
+      (effects (font (size 1.27 1.27)) hide)
+    )
