File: mainboard/2layer/kicad/config_selection.kicad_sch (KiCad schematic)
At the start: 17 parts, among them U17 74LS00, U35 74LS86, U36 74LS74, U52 74LS11, U53 74LS04, U54 74LS00, U55 74LS00, U56 74LS42

Commit message: Fixes for PCB DRC: trace clearance, footprints, board edges
Parts:
- D1, D2, D3: footprint Diode_THT:D_DO-35_SOD27_P7.62mm_Horizontal -> Cobra_original:D_DO-35_SOD27_P7.62mm_Horizontal
Changed lines of the file:
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@@
       (effects (font (size 1.27 1.27)))
     )
-    (property "Footprint" "Diode_THT:D_DO-35_SOD27_P7.62mm_Horizontal" (at 131.445 133.985 0)
+    (property "Footprint" "Cobra_original:D_DO-35_SOD27_P7.62mm_Horizontal" (at 131.445 133.985 0)
       (effects (font (size 1.27 1.27)) hide)
     )
@@
       (effects (font (size 1.27 1.27)))
     )
-    (property "Footprint" "Diode_THT:D_DO-35_SOD27_P7.62mm_Horizontal" (at 131.445 146.685 0)
+    (property "Footprint" "Cobra_original:D_DO-35_SOD27_P7.62mm_Horizontal" (at 131.445 146.685 0)
       (effects (font (size 1.27 1.27)) hide)
     )
@@
       (effects (font (size 1.27 1.27)) (justify left))
     )
-    (property "Footprint" "Diode_THT:D_DO-35_SOD27_P7.62mm_Horizontal" (at 80.01 149.86 0)
-      (effects (font (size 1.27 1.27)) hide)
-    )
+    (property "Footprint" "Cobra_original:D_DO-35_SOD27_P7.62mm_Horizontal" (at 80.01 149.86 0)
+      (effects (font (size 1.27 1.27)) hide)
+    )
