File: mainboard/2layer/kicad/video_generator.kicad_sch (KiCad schematic)
At the start: 40 parts, among them J1 Conn_01x10, Q2 2N2219, U77 74LS95, U78 74LS95, U80 74LS157, U81 74LS95, U82 74LS95, U83 74LS95, U85 74LS157, U86 CDB407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

Commit message: Fixes for PCB DRC: trace clearance, footprints, board edges
Parts:
- D4, DBR1, DBR2, DBR3, DBR4, DBR5: footprint Diode_THT:D_DO-35_SOD27_P7.62mm_Horizontal -> Cobra_original:D_DO-35_SOD27_P7.62mm_Horizontal
- J1: footprint Connector_PinHeader_2.54mm:PinHeader_1x10_P2.54mm_Vertical -> Cobra_original:PinHeader_1x10_P2.54mm_Vertical
Changed lines of the file:
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@@
       (effects (font (size 1.27 1.27)) hide)
     )
-    (property "Footprint" "Diode_THT:D_DO-35_SOD27_P7.62mm_Horizontal" (at 81.28 229.235 0)
+    (property "Footprint" "Cobra_original:D_DO-35_SOD27_P7.62mm_Horizontal" (at 81.28 229.235 0)
       (effects (font (size 1.27 1.27)) hide)
     )
@@
       (effects (font (size 1.27 1.27)) hide)
     )
-    (property "Footprint" "Diode_THT:D_DO-35_SOD27_P7.62mm_Horizontal" (at 81.28 233.045 0)
+    (property "Footprint" "Cobra_original:D_DO-35_SOD27_P7.62mm_Horizontal" (at 81.28 233.045 0)
       (effects (font (size 1.27 1.27)) hide)
     )
@@
       (effects (font (size 1.27 1.27)) hide)
     )
-    (property "Footprint" "Diode_THT:D_DO-35_SOD27_P7.62mm_Horizontal" (at 62.23 233.045 0)
+    (property "Footprint" "Cobra_original:D_DO-35_SOD27_P7.62mm_Horizontal" (at 62.23 233.045 0)
       (effects (font (size 1.27 1.27)) hide)
     )
@@
       (effects (font (size 1.27 1.27)) hide)
     )
-    (property "Footprint" "Diode_THT:D_DO-35_SOD27_P7.62mm_Horizontal" (at 62.23 236.855 0)
+    (property "Footprint" "Cobra_original:D_DO-35_SOD27_P7.62mm_Horizontal" (at 62.23 236.855 0)
       (effects (font (size 1.27 1.27)) hide)
     )
@@
       (effects (font (size 1.27 1.27)) hide)
     )
-    (property "Footprint" "Diode_THT:D_DO-35_SOD27_P7.62mm_Horizontal" (at 62.23 240.665 0)
+    (property "Footprint" "Cobra_original:D_DO-35_SOD27_P7.62mm_Horizontal" (at 62.23 240.665 0)
       (effects (font (size 1.27 1.27)) hide)
     )
@@
       (effects (font (size 1.27 1.27)))
     )
-    (property "Footprint" "Diode_THT:D_DO-35_SOD27_P7.62mm_Horizontal" (at 128.27 172.085 0)
+    (property "Footprint" "Cobra_original:D_DO-35_SOD27_P7.62mm_Horizontal" (at 128.27 172.085 0)
       (effects (font (size 1.27 1.27)) hide)
     )
@@
       (effects (font (size 1.27 1.27)) hide)
     )
-    (property "Footprint" "Connector_PinHeader_2.54mm:PinHeader_1x10_P2.54mm_Vertical" (at 190.5 187.96 0)
-      (effects (font (size 1.27 1.27)) hide)
-    )
+    (property "Footprint" "Cobra_original:PinHeader_1x10_P2.54mm_Vertical" (at 190.5 187.96 0)
+      (effects (font (size 1.27 1.27)) hide)
+    )
